File: TPS65217A Evaluation Board.brd (EAGLE design)
At the start: 160 x 100 mm, 39 parts, among them U1 TPS65217ARSLR

Commit message: Add files via upload
Parts:
- removed PB_IN: TEST_TESTPOINT, marius:TEST_TESTPOINT
- moved 1V2 54.5 mm to (80.7, 47.3)
- moved 3V3 50.1 mm to (72.2, 34.2)
- moved SDA 44.6 mm to (71.8, 58.7), turned to 90 degrees
- moved SCL 42.9 mm to (69.6, 58.7), turned to 90 degrees
- moved NRESET 41.8 mm to (66.0, 58.7), turned to 90 degrees
- moved 1V8 40.7 mm to (62.7, 33.9)
- moved LDO3V3 40.4 mm to (60.1, 58.5), turned to 90 degrees
- moved LDO1V8 40.4 mm to (61.8, 58.5), turned to 90 degrees
- moved SYS 32.4 mm to (60.1, 46.3), turned to 270 degrees
- moved MUX 25.0 mm to (51.8, 38.7), turned to 180 degrees
- moved PWR_EN 23.1 mm to (50.7, 42.3)
- moved CN1 3.50 mm to (52.1, 53.3)
- moved C3 0.75 mm to (60.8, 49.4)
Connections:
- removed net PB_IN: PB_IN.1, U1.25
Routing:
- net VBAT: track 17.0 -> 0.70 mm
- net PWR_EN: track 0.00 -> 11.1 mm
- net GND: track 13.2 -> 5.00 mm
- net MUX_OUT: track 12.0 -> 12.5 mm
- net SYS: vias 1 -> 8
- added copper zone on layer 1, net VBAT
