File: TPS65217A Evaluation Board.brd (EAGLE design)
At the start: 38.5 x 29 mm, 39 parts, among them U1 TPS65217ARSLR

Commit message: V1
Parts:
- renumbered U1 to GND
Routing:
- net GND: vias 20 -> 29
Changed lines of the file:
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@@
 <vertex x="44.29" y="61.03"/>
 </polygon>
+<wire x1="44.25" y1="32" x2="44.25" y2="61" width="0" layer="20"/>
+<wire x1="44.25" y1="61" x2="82.75" y2="61" width="0" layer="20"/>
+<wire x1="82.75" y1="61" x2="82.75" y2="32" width="0" layer="20"/>
+<wire x1="82.75" y1="32" x2="44.25" y2="32" width="0" layer="20"/>
 </plain>
 <attributes>
@@
 </autorouter>
 <elements>
-<element name="U1" library="iframe" package="RSL48_4P05X4P05" value="TPS65217ARSLR" x="66.04" y="46.99" smashed="yes">
+<element name="GND" library="iframe" package="RSL48_4P05X4P05" value="TPS65217ARSLR" x="66.04" y="46.99" smashed="yes">
 <attribute name="MANUFACTURER_PART_NUMBER" value="TPS65217ARSLR" x="83.82" y="41.91" size="1.778" layer="27" display="off"/>
 <attribute name="NAME" x="62.7634" y="46.355" size="1.27" layer="25" ratio="6" rot="SR0"/>
@@
 <signals>
 <signal name="VUSB">
-<contactref element="U1" pad="12"/>
+<contactref element="GND" pad="12"/>
 <contactref element="C5" pad="2"/>
 <wire x1="56.14" y1="41.66" x2="56.4024" y2="41.3976" width="0.2" layer="1"/>
@@
 </signal>
 <signal name="VBAT">
-<contactref element="U1" pad="5"/>
-<contactref element="U1" pad="4"/>
+<contactref element="GND" pad="5"/>
+<contactref element="GND" pad="4"/>
 <contactref element="C3" pad="2"/>
-<contactref element="U1" pad="6"/>
+<contactref element="GND" pad="6"/>
 <contactref element="CN1" pad="2"/>
 <polygon width="0.127" layer="1" thermals="no">
@@
 </signal>
 <signal name="SCL">
-<contactref element="U1" pad="28"/>
+<contactref element="GND" pad="28"/>
 <contactref element="R6" pad="1"/>
 <contactref element="SCL" pad="1"/>
@@
 </signal>
 <signal name="SDA">
-<contactref element="U1" pad="27"/>
+<contactref element="GND" pad="27"/>
 <contactref element="R5" pad="1"/>
 <contactref element="SDA" pad="1"/>
@@
 </signal>
 <signal name="LDO4">
-<contactref element="U1" pad="43"/>
+<contactref element="GND" pad="43"/>
 <contactref element="C23" pad="2"/>
 <wire x1="65.84" y1="49.965" x2="65.84" y2="50.59819375" width="0.2" layer="1"/>
@@
 </signal>
 <signal name="LDO3">
-<contactref element="U1" pad="40"/>
+<contactref element="GND" pad="40"/>
 <contactref element="C22" pad="2"/>
 <wire x1="68.39" y1="53.61" x2="68.39" y2="52.89" width="0.2" layer="1"/>
@@
 </signal>
 <signal name="MUX_OUT">
-<contactref element="U1" pad="16"/>
+<contactref element="GND" pad="16"/>
 <contactref element="C9" pad="2"/>
 <contactref element="MUX" pad="1"/>
@@
 </signal>
 <signal name="SYS">
-<contactref element="U1" pad="32"/>
+<contactref element="GND" pad="32"/>
 <contactref element="C10" pad="2"/>
-<contactref element="U1" pad="21"/>
+<contactref element="GND" pad="21"/>
 <contactref element="C20" pad="2"/>
-<contactref element="U1" pad="22"/>
+<contactref element="GND" pad="22"/>
 <contactref element="C19" pad="2"/>
-<contactref element="U1" pad="2"/>
+<contactref element="GND" pad="2"/>
 <contactref element="C6" pad="2"/>
-<contactref element="U1" pad="39"/>
-<contactref element="U1" pad="42"/>
-<contactref element="U1" pad="7"/>
-<contactref element="U1" pad="8"/>
+<contactref element="GND" pad="39"/>
+<contactref element="GND" pad="42"/>
+<contactref element="GND" pad="7"/>
+<contactref element="GND" pad="8"/>
 <contactref element="C4" pad="2"/>
 <contactref element="C16" pad="2"/>
@@
 </signal>
 <signal name="VDCDC3">
-<contactref element="U1" pad="29"/>
+<contactref element="GND" pad="29"/>
 <contactref element="R8" pad="1"/>
 <contactref element="R9" pad="1"/>
@@
 </signal>
 <signal name="LDO3V3">
-<contactref element="U1" pad="1"/>
+<contactref element="GND" pad="1"/>
 <contactref element="LDO3V3" pad="1"/>
 <wire x1="63.065" y1="49.19" x2="63.065" y2="50.685" width="0.254" layer="1"/>
@@
 </signal>
 <signal name="LDO1V8">
-<contactref element="U1" pad="3"/>
-<contactref element="U1" pad="18"/>
+<contactref element="GND" pad="3"/>
+<contactref element="GND" pad="18"/>
 <contactref element="LDO1V8" pad="1"/>
 <wire x1="65.84" y1="44.015" x2="65.84" y2="44.5" width="0.2" layer="1"/>
@@
 </signal>
 <signal name="L2">
-<contactref element="U1" pad="23"/>
+<contactref element="GND" pad="23"/>
 <contactref element="L2" pad="P$2"/>
 <polygon width="0.1524" layer="1" thermals="no">
@@
 </signal>
 <signal name="L1">
-<contactref element="U1" pad="20"/>
+<contactref element="GND" pad="20"/>
 <contactref element="L1" pad="P$2"/>
 <polygon width="0.15" layer="1" thermals="no">
@@
 </signal>
 <signal name="NWAKEUP">
-<contactref element="U1" pad="13"/>
+<contactref element="GND" pad="13"/>
 <contactref element="R10" pad="1"/>
 <wire x1="56.06" y1="36.69" x2="55.56" y2="36.69" width="0.1524" layer="1"/>
@@
 </signal>
 <signal name="INT_LDO">
-<contactref element="U1" pad="48"/>
+<contactref element="GND" pad="48"/>
 <contactref element="C7" pad="2"/>
 <wire x1="63.84" y1="49.965" x2="63.84" y2="50.91" width="0.2" layer="1"/>
@@
 </signal>
 <signal name="PWR_EN">
-<contactref element="U1" pad="9"/>
+<contactref element="GND" pad="9"/>
 <contactref element="PWR_EN" pad="1"/>
 <wire x1="63.065" y1="45.99" x2="62.49" y2="45.99" width="0.1524" layer="1"/>
@@
 </signal>
 <signal name="NRESET">
-<contactref element="U1" pad="44"/>
+<contactref element="GND" pad="44"/>
 <contactref element="NRESET" pad="1"/>
 <wire x1="65.44" y1="49.965" x2="65.44" y2="50.49981875" width="0.2" layer="1"/>
@@
 </signal>
 <signal name="BYPASS">
-<contactref element="U1" pad="47"/>
+<contactref element="GND" pad="47"/>
 <contactref element="C21" pad="2"/>
 <wire x1="64.24" y1="49.965" x2="64.24" y2="51.0756875" width="0.2" layer="1"/>
@@
 </signal>
 <signal name="NINT">
-<contactref element="U1" pad="45"/>
+<contactref element="GND" pad="45"/>
 <contactref element="R11" pad="1"/>
 <wire x1="65.22" y1="53.61" x2="65.22" y2="53.0036125" width="0.2" layer="1"/>
@@
 <signal name="BATTERYTEMP_10KNTC">
 <contactref element="R7" pad="2"/>
-<contactref element="U1" pad="11"/>
+<contactref element="GND" pad="11"/>
 <wire x1="63.065" y1="45.19" x2="61.44" y2="45.19" width="0.2" layer="1"/>
 <wire x1="57.5" y1="43.25" x2="56.19" y2="43.25" width="0.2" layer="1"/>
@@
 </signal>
 <signal name="L3">
-<contactref element="U1" pad="31"/>
+<contactref element="GND" pad="31"/>
 <contactref element="L3" pad="P$2"/>
 <wire x1="75.462" y1="47.117" x2="75.389" y2="47.19" width="0.6096" layer="1"/>
@@
 <contactref element="C21" pad="1"/>
 <contactref element="C7" pad="1"/>
-<contactref element="U1" pad="30"/>
-<contactref element="U1" pad="41"/>
-<contactref element="U1" pad="49"/>
+<contactref element="GND" pad="30"/>
+<contactref element="GND" pad="41"/>
+<contactref element="GND" pad="49"/>
 <contactref element="R9" pad="2"/>
 <contactref element="C9" pad="1"/>
@@
 <wire x1="66.64" y1="49.36" x2="66.64" y2="49.965" width="0.2032" layer="1"/>
 <wire x1="66.75" y1="49.25" x2="66.64" y2="49.36" width="0.2032" layer="1"/>
-<wire x1="68.336" y1="46.9847875" x2="66.04" y2="46.99" width="0" layer="19" extent="1-1"/>
+<via x="67.25" y="45.75" extent="1-16" drill="0.35"/>
+<via x="66" y="45.75" extent="1-16" drill="0.35"/>
+<via x="64.75" y="45.75" extent="1-16" drill="0.35"/>
+<via x="64.75" y="47" extent="1-16" drill="0.35"/>
+<via x="64.75" y="48.25" extent="1-16" drill="0.35"/>
+<via x="66" y="48.25" extent="1-16" drill="0.35"/>
+<via x="66" y="47" extent="1-16" drill="0.35"/>
+<via x="67.25" y="47" extent="1-16" drill="0.35"/>
+<via x="67.25" y="48.25" extent="1-16" drill="0.35"/>
 </signal>
 <signal name="3V3">
 <contactref element="R6" pad="2"/>
 <contactref element="R5" pad="2"/>
-<contactref element="U1" pad="24"/>
+<contactref element="GND" pad="24"/>
 <contactref element="L2" pad="P$1"/>
-<contactref element="U1" pad="14"/>
+<contactref element="GND" pad="14"/>
 <contactref element="R10" pad="2"/>
 <contactref element="R11" pad="2"/>
@@
 </signal>
 <signal name="1V8">
-<contactref element="U1" pad="19"/>
+<contactref element="GND" pad="19"/>
 <contactref element="L1" pad="P$1"/>
 <contactref element="1V8" pad="1"/>

Commit message: V1
Parts:
- added LDO3, LDO4: TEST_TESTPOINT, marius:TEST_TESTPOINT
Connections:
- net LDO3: now also LDO3.1
- net LDO4: now also LDO4.1
Routing:
- net LDO3: track 4.20 -> 11.3 mm
- net LDO4: track 4.09 -> 8.98 mm
Changed lines of the file:
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@@
 <drawing>
 <settings>
-<setting alwaysvectorfont="no"/>
+<setting alwaysvectorfont="yes"/>
 <setting verticaltext="up"/>
 </settings>
@@
 </layers>
 <board>
+<fusionsync huburn="a.cGVyc29uYWw6dWUyOTQ3ODVk" projecturn="a.cGVyc29uYWw6dWUyOTQ3ODVkIzIwMTgwODE1MTQ0MTI2NzUx" f3durn="urn:adsk.wipprod:dm.lineage:44Vuc7aUT0mz-DZkzW1-Yg" pcbguid="8762834f-3f7f-4e23-9605-112ef1adf8f7" lastpulledtime="" lastsyncedchangeguid="2bec2dfb-6afe-e8ac-4bb2-5b1c546bf32b"/>
 <plain>
 <polygon width="0.1524" layer="46">
@@
 <attribute name="VALUE" x="42.15" y="42.5516" size="1.27" layer="27" font="vector" ratio="13" rot="SR270"/>
 </element>
+<element name="LDO4" library="marius" package="TEST_TESTPOINT" package3d_urn="urn:adsk.eagle:package:5911110/1" value="TEST_TESTPOINT" x="68" y="58" smashed="yes">
+<attribute name="NAME" x="68.635" y="58" size="0.7" layer="25" align="center-left"/>
+<attribute name="X" value="X" x="68" y="58" size="1.778" layer="27" display="off"/>
+</element>
+<element name="LDO3" library="marius" package="TEST_TESTPOINT" package3d_urn="urn:adsk.eagle:package:5911110/1" value="TEST_TESTPOINT" x="72.25" y="58" smashed="yes">
+<attribute name="NAME" x="72.885" y="58" size="0.7" layer="25" align="center-left"/>
+<attribute name="X" value="X" x="72.25" y="58" size="1.778" layer="27" display="off"/>
+</element>
 </elements>
 <signals>
@@
 <wire x1="66.78" y1="52.78" x2="66.78" y2="53.61" width="0.2" layer="1"/>
 <wire x1="65.7788" y1="51.7788" x2="66.78" y2="52.78" width="0.2" layer="1"/>
+<contactref element="LDO4" pad="1"/>
+<wire x1="68" y1="57.10815" x2="68" y2="58" width="0.1524" layer="1"/>
+<wire x1="66.78" y1="53.61" x2="67.6614" y2="54.4914" width="0.1524" layer="1"/>
+<wire x1="67.6614" y1="54.4914" x2="67.6614" y2="56.76955" width="0.1524" layer="1"/>
+<wire x1="67.6614" y1="56.76955" x2="68" y2="57.10815" width="0.1524" layer="1"/>
 </signal>
 <signal name="LDO3">
@@
 <wire x1="68.39" y1="52.89" x2="67.1306" y2="51.6306" width="0.2" layer="1"/>
 <wire x1="67.1306" y1="51.6306" x2="67.1306" y2="50.98879375" width="0.2" layer="1"/>
+<contactref element="LDO3" pad="1"/>
+<wire x1="72.25" y1="57.47" x2="72.25" y2="58" width="0.1524" layer="1"/>
+<wire x1="71.6368" y1="56.8568" x2="72.25" y2="57.47" width="0.1524" layer="1"/>
+<wire x1="68.39" y1="53.61" x2="69.1314" y2="54.3514" width="0.1524" layer="1"/>
+<wire x1="69.1314" y1="54.3514" x2="69.1314" y2="56.23955" width="0.1524" layer="1"/>
+<wire x1="69.1314" y1="56.23955" x2="69.74865" y2="56.8568" width="0.1524" layer="1"/>
+<wire x1="69.74865" y1="56.8568" x2="71.6368" y2="56.8568" width="0.1524" layer="1"/>
 </signal>
 <signal name="MUX_OUT">
@@
 <wire x1="71.5" y1="56.25" x2="77.75" y2="56.25" width="0.2" layer="16"/>
 <wire x1="77.75" y1="56.25" x2="77.75" y2="38.5" width="0.2" layer="16"/>
-<wire x1="77.75" y1="38.5" x2="74.5" y2="35.25" width="0.2" layer="16"/>
-<wire x1="74.5" y1="35.25" x2="70.25" y2="35" width="0.2" layer="16"/>
+<wire x1="77.75" y1="38.5" x2="74.25" y2="35" width="0.2" layer="16"/>
+<wire x1="74.25" y1="35" x2="70.25" y2="35" width="0.2" layer="16"/>
 <wire x1="69.91" y1="55.31" x2="69.91" y2="56.16" width="0.2" layer="1"/>
 <wire x1="69.91" y1="56.16" x2="70" y2="56.25" width="0.2" layer="1"/>
@@
 </note>
 <note version="8.3" severity="warning">
+Since Version 8.3, EAGLE supports Fusion synchronisation.
+This feature will not be available in this version and saving
+the document will break the link to the Fusion PCB feature.
+</note>
+<note version="8.3" severity="warning">
